Commit message: Changing name of gazebo colors for pantilt robot

File: pantilt_description/model/pantilt_gazebo.urdf.xacro (robot description, xacro)
@@ -47,5 +47,5 @@
 					<mesh filename="package://pantilt_description/meshes/bati.stl"/>
 				</geometry>
-				<material name="DarkGrey" />
+				<material name="PantiltDarkGrey" />
 			</visual>
 			<!--visual>
@@ -80,5 +80,5 @@
 					<mesh filename="package://pantilt_description/meshes/P1.stl"/>
 				</geometry>
-				<material name="DarkGrey" />
+				<material name="PantiltDarkGrey" />
 			</visual>
 			<!--visual>
@@ -119,5 +119,5 @@
 					<mesh filename="package://pantilt_description/meshes/P2.stl"/>
 				</geometry>
-				<material name="DarkGrey" />
+				<material name="PantiltDarkGrey" />
 			</visual>
 			<!--visual>
@@ -160,5 +160,5 @@
 					<mesh filename="package://pantilt_description/meshes/cam.stl"/>
 				</geometry>
-				<material name="LightGrey" />
+				<material name="PantiltLightGrey" />
 			</visual>
 		</link>
@@ -193,5 +193,5 @@
 					<mesh filename="package://pantilt_description/meshes/cam.stl"/>
 				</geometry>
-				<material name="LightGrey" />
+				<material name="PantiltLightGrey" />
 			</visual>
 		</link>

File: pantilt_description/model/pantilt_materials.xacro (robot description, xacro)
@@ -1,11 +1,11 @@
 <?xml version="1.0"?>
 <robot xmlns:xacro="http://ros.org/wiki/xacro">
-  <material name="DarkGrey">
+  <material name="PantiltDarkGrey">
     <color rgba="0.3 0.3 0.3 1.0"/>
   </material>
-  <material name="LightGrey">
+  <material name="PantiltLightGrey">
     <color rgba="0.8 0.8 0.8 1.0"/>
   </material>
-  <material name="Black">
+  <material name="PantiltBlack">
     <color rgba="0 0 0 1.0"/>
   </material>
