Commit message: Adding bi manual (sh lh et rh) definition, gazebo, launch

File: platform_gazebo/robot/platform_robot_shadow_hands.urdf.xacro (robot description, xacro)
@@ -40,5 +40,5 @@
  <xacro:include filename="$(find sr_description)/hand/xacro/full_hand.urdf.xacro"/>
  <xacro:include filename="$(find platform_gazebo)/robot/sr/gazebo.urdf.xacro"/>
- <xacro:macro name="shadow_hand" params="parent name namespace prefix *origin">
+ <xacro:macro name="shadow_hand" params="parent name prefix *origin">
 		<joint name="${parent}_${name}_hand_joint" type="fixed">
 		  <parent link="${parent}" />
@@ -50,13 +50,14 @@
  </xacro:macro>
 <!--<xacro:if value="$(arg use_right_hand)">-->
-   <xacro:shadow_hand parent="kuka_lwr_right_7_link" name="shadow_hand_right" namespace="shadow_hand_right" prefix="rh">
+   <xacro:shadow_hand parent="kuka_lwr_right_7_link" name="sh_rh" prefix="rh">
 		<origin xyz="0 0 0" rpy="0 0 0"/>
    </xacro:shadow_hand>
-	<xacro:sr_gazebo name="sr_rh" namespace="shadow_hand"/>
+   <xacro:sr_gazebo name="sr_rh" namespace="/rh"/>
 <!--</xacro:if>-->
-<!--<xacro:if value="$(arg use_left_hand)">
-  <xacro:shadow_hand parent="kuka_lwr_left_7_link" name="shadow_hand_left" namespace="shadow_hand_left" prefix="lh">
+<!--<xacro:if value="$(arg use_left_hand)">-->
+  <xacro:shadow_hand parent="kuka_lwr_left_7_link" name="sh_lh" prefix="lh">
 		<origin xyz="0 0 0" rpy="0 0 ${pi}"/>
-   </xacro:shadow_hand>
-</xacro:if>-->
+  </xacro:shadow_hand>
+  <xacro:sr_gazebo name="sr_lh" namespace="/lh"/>
+<!--</xacro:if>-->
 </robot>

File: platform_gazebo/robot/sr/gazebo.urdf.xacro (robot description, xacro)
@@ -4,6 +4,6 @@
 		<gazebo>
 			<plugin name="${name}_gazebo_ros_control" filename="libgazebo_ros_control.so">
+				<robotSimType>sr_gazebo_sim/SrGazeboHWSim</robotSimType>
 				<robotNamespace>${namespace}</robotNamespace>
-				<robotSimType>sr_gazebo_sim/SrGazeboHWSim</robotSimType>
 			</plugin>
 		</gazebo>
