Commit message: Adding first version for barrett hand

File: platform_gazebo/robot/platform_robot_with_hands.urdf.xacro (robot description, xacro)
@@ -49,15 +49,36 @@
 						  ubi="false" eli="false" reflect="1.0" prefix="${prefix}_" lf="true" />
  </xacro:macro>
-<xacro:if value="$(arg use_right_sh)">
+ <xacro:if value="$(arg use_right_sh)">
    <xacro:shadow_hand parent="kuka_lwr_right_7_link" name="rsh" prefix="rh">
 		<origin xyz="0 0 0" rpy="0 0 0"/>
    </xacro:shadow_hand>
    <xacro:sr_gazebo name="rsh_gazebo" namespace="/rsh"/>
-</xacro:if>
-<xacro:if value="$(arg use_left_sh)">
+ </xacro:if>
+ <xacro:if value="$(arg use_left_sh)">
   <xacro:shadow_hand parent="kuka_lwr_left_7_link" name="lsh" prefix="lh">
 		<origin xyz="0 0 0" rpy="0 0 ${pi}"/>
   </xacro:shadow_hand>
   <xacro:sr_gazebo name="lsh_gazebo" namespace="/lsh"/>
-</xacro:if>
+ </xacro:if>
+ <!-- Create Barrett Hand -->
+ <!-- Available choices: bh282.urdf.xacro, bh280.urdf.xacro -->
+ <xacro:include filename="$(find barrett_hand_description)/urdf/bh280.urdf.xacro" />
+ <xacro:include filename="$(find platform_gazebo)/robot/barrett_hand/bh_gazebo.urdf.xacro"/>
+ <xacro:macro name="barrett_hand" params="parent name *origin">
+		<xacro:bhand_macro name="${name}" parent="${parent}">
+		    <insert_block name="origin"/>
+	    </xacro:bhand_macro>
+ </xacro:macro>
+ <xacro:if value="$(arg use_right_bh)">
+   <xacro:barrett_hand parent="kuka_lwr_right_7_link" name="rbh" >
+		<origin xyz="0 0 0" rpy="0 0 0"/>
+   </xacro:barrett_hand>
+   <xacro:bh_ros_control_gazebo name="rbh" namespace="/rbh"/>
+ </xacro:if>
+ <xacro:if value="$(arg use_left_bh)">
+   <xacro:barrett_hand parent="kuka_lwr_left_7_link" name="lbh"  >
+		<origin xyz="0 0 0" rpy="0 0 ${pi}"/>
+   </xacro:barrett_hand>
+   <xacro:bh_ros_control_gazebo name="lbh" namespace="/lbh"/>
+ </xacro:if>
 </robot>

Commit message: Set good rotation for right and left shadow hand

File: platform_gazebo/robot/platform_robot_with_hands.urdf.xacro (robot description, xacro)
@@ -17,9 +17,9 @@
   <!-- Create Kuka LWR Right -->
   <xacro:kuka_lwr parent="trunk_link" name="kuka_lwr_right">
-	<origin xyz="-0.17 0 1.45" rpy="0 ${pi/2.0} ${pi}"/>
+	<origin xyz="0.17 0 1.45" rpy="0 ${pi/2.0} 0"/>
   </xacro:kuka_lwr>
   <!-- Create Kuka LWR Left -->
   <xacro:kuka_lwr parent="trunk_link" name="kuka_lwr_left">
-	<origin xyz="0.17 0 1.45" rpy="0 ${pi/2.0} 0"/>
+	<origin xyz="-0.17 0 1.45" rpy="0 ${pi/2.0} ${pi}"/>
   </xacro:kuka_lwr>
  <!-- Create Gazebo Kuka Right -->
@@ -40,5 +40,5 @@
  <xacro:include filename="$(find sr_description)/hand/xacro/full_hand.urdf.xacro"/>
  <xacro:include filename="$(find platform_gazebo)/robot/sr/sr_gazebo.urdf.xacro"/>
- <xacro:macro name="shadow_hand" params="parent name prefix *origin">
+ <xacro:macro name="shadow_hand" params="parent name prefix reflect *origin">
 		<joint name="${parent}_${name}_hand_joint" type="fixed">
 		  <parent link="${parent}" />
@@ -47,15 +47,15 @@
 		</joint>
 		<xacro:shadowhand muscletrans="false" muscle="false" bio="false" bt_sp="false"
-						  ubi="false" eli="false" reflect="1.0" prefix="${prefix}_" lf="true" />
+						  ubi="false" eli="false" reflect="${reflect}" prefix="${prefix}_" lf="true" />
  </xacro:macro>
  <xacro:if value="$(arg use_right_sh)">
-   <xacro:shadow_hand parent="kuka_lwr_right_7_link" name="rsh" prefix="rh">
-		<origin xyz="0 0 0" rpy="0 0 0"/>
+   <xacro:shadow_hand parent="kuka_lwr_right_7_link" name="rsh" prefix="rh" reflect="1.0">
+		<origin xyz="0 0 0" rpy="0 0 ${pi}"/>
    </xacro:shadow_hand>
    <xacro:sr_gazebo name="rsh_gazebo" namespace="/rsh"/>
  </xacro:if>
  <xacro:if value="$(arg use_left_sh)">
-   <xacro:shadow_hand parent="kuka_lwr_left_7_link" name="lsh" prefix="lh">
-		<origin xyz="0 0 0" rpy="0 0 ${pi}"/>
+   <xacro:shadow_hand parent="kuka_lwr_left_7_link" name="lsh" prefix="lh" reflect="-1.0">
+		<origin xyz="0 0 0" rpy="0 0 0"/>
    </xacro:shadow_hand>
    <xacro:sr_gazebo name="lsh_gazebo" namespace="/lsh"/>
@@ -63,21 +63,16 @@
  <!-- Create Barrett Hand -->
  <!-- Available choices: bh282.urdf.xacro, bh280.urdf.xacro -->
- <xacro:include filename="$(find barrett_hand_description)/urdf/bh280.urdf.xacro" />
+ <xacro:include filename="$(find barrett_hand_description)/urdf/bh280.urdf.xacro"/>
  <xacro:include filename="$(find platform_gazebo)/robot/barrett_hand/bh_gazebo.urdf.xacro"/>
- <xacro:macro name="barrett_hand" params="parent name *origin">
-		<xacro:bhand_macro name="${name}" parent="${parent}">
-		    <insert_block name="origin"/>
-	    </xacro:bhand_macro>
- </xacro:macro>
  <xacro:if value="$(arg use_right_bh)">
-   <xacro:barrett_hand parent="kuka_lwr_right_7_link" name="rbh" >
-		<origin xyz="0 0 0" rpy="0 0 0"/>
-   </xacro:barrett_hand>
+	<xacro:bhand_macro name="rbh" parent="kuka_lwr_right_7_link">
+		<origin xyz="0 0 0" rpy="0 0 0" />
+	</xacro:bhand_macro>
    <xacro:bh_ros_control_gazebo name="rbh_gazebo" namespace="/rbh"/>
  </xacro:if>
  <xacro:if value="$(arg use_left_bh)">
-   <xacro:barrett_hand parent="kuka_lwr_left_7_link" name="lbh" >
-		<origin xyz="0 0 0" rpy="0 0 ${pi}"/>
-   </xacro:barrett_hand>
+	<xacro:bhand_macro name="lbh" parent="kuka_lwr_left_7_link">
+		<origin xyz="0 0 0" rpy="0 0 ${pi}" />
+	</xacro:bhand_macro>
    <xacro:bh_ros_control_gazebo name="lbh_gazebo" namespace="/lbh"/>
  </xacro:if>
