Commit message: Adding simple version based on all joint controllers

File: platform_gazebo/robot/lbh_barrett_hand.urdf.xacro (robot description, xacro)
@@ -5,13 +5,8 @@
   <!-- Create Barrett Hand -->
   <!-- Available choices: bh282.urdf.xacro, bh280.urdf.xacro -->
-  <xacro:include filename="$(find barrett_hand_description)/urdf/bh280.urdf.xacro" />
-  <xacro:macro name="barrett_hand" params="parent name *origin">
-		<xacro:bhand_macro name="${name}" parent="${parent}">
-		    <insert_block name="origin"/>
-	    </xacro:bhand_macro>
-  </xacro:macro>
+  <xacro:include filename="$(find barrett_hand_description)/urdf/ip_bh280.urdf.xacro" />
   <link name="kuka_lwr_left_7_link"/>
-  <xacro:barrett_hand parent="kuka_lwr_left_7_link" name="lbh"  >
-	<origin xyz="0 0 0" rpy="0 0 ${pi}"/>
-  </xacro:barrett_hand>
+  <xacro:bhand_macro name="lbh" namespace="/lbh" parent="kuka_lwr_left_7_link">
+		<origin xyz="0 0 0" rpy="0 0 ${pi}" />
+  </xacro:bhand_macro>
 </robot>

File: platform_gazebo/robot/platform_robot_with_hands.urdf.xacro (robot description, xacro)
@@ -63,17 +63,17 @@
  <!-- Create Barrett Hand -->
  <!-- Available choices: bh282.urdf.xacro, bh280.urdf.xacro -->
- <xacro:include filename="$(find barrett_hand_description)/urdf/bh280.urdf.xacro"/>
- <xacro:include filename="$(find platform_gazebo)/robot/barrett_hand/bh_gazebo.urdf.xacro"/>
+ <xacro:include filename="$(find barrett_hand_description)/urdf/ip_bh280.urdf.xacro"/>
+ <!--<xacro:include filename="$(find platform_gazebo)/robot/barrett_hand/bh_gazebo.urdf.xacro"/>-->
  <xacro:if value="$(arg use_right_bh)">
-	<xacro:bhand_macro name="rbh" parent="kuka_lwr_right_7_link">
+	<xacro:bhand_macro name="rbh" namespace="/rbh" parent="kuka_lwr_right_7_link">
 		<origin xyz="0 0 0" rpy="0 0 0" />
 	</xacro:bhand_macro>
-   <xacro:bh_ros_control_gazebo name="rbh_gazebo" namespace="/rbh"/>
+   <!--<xacro:bh_ros_control_gazebo name="rbh_gazebo" namespace="/rbh"/>-->
  </xacro:if>
  <xacro:if value="$(arg use_left_bh)">
-	<xacro:bhand_macro name="lbh" parent="kuka_lwr_left_7_link">
+	<xacro:bhand_macro name="lbh" namespace="/lbh" parent="kuka_lwr_left_7_link">
 		<origin xyz="0 0 0" rpy="0 0 ${pi}" />
 	</xacro:bhand_macro>
-   <xacro:bh_ros_control_gazebo name="lbh_gazebo" namespace="/lbh"/>
+   <!--<xacro:bh_ros_control_gazebo name="lbh_gazebo" namespace="/lbh"/>-->
  </xacro:if>
 </robot>

File: platform_gazebo/robot/rbh_barrett_hand.urdf.xacro (robot description, xacro)
@@ -3,13 +3,8 @@
   <!-- Create Barrett Hand -->
   <!-- Available choices: bh282.urdf.xacro, bh280.urdf.xacro -->
-  <xacro:include filename="$(find barrett_hand_description)/urdf/bh280.urdf.xacro" />
-  <xacro:macro name="barrett_hand" params="parent name *origin">
-		<xacro:bhand_macro name="${name}" parent="${parent}">
-		    <insert_block name="origin"/>
-	    </xacro:bhand_macro>
-  </xacro:macro>
+  <xacro:include filename="$(find barrett_hand_description)/urdf/ip_bh280.urdf.xacro" />
   <link name="kuka_lwr_right_7_link"/>
-  <xacro:barrett_hand parent="kuka_lwr_right_7_link" name="rbh"  >
-	<origin xyz="0 0 0" rpy="0 0 0"/>
-  </xacro:barrett_hand>
+  <xacro:bhand_macro name="rbh" namespace="/rbh" parent="kuka_lwr_right_7_link">
+		<origin xyz="0 0 0" rpy="0 0 0" />
+  </xacro:bhand_macro>
 </robot>
