Commit message: Adding ip version of barrettt hand description

File: effectors/barrett_hand/barrett_hand_common/barrett_hand_description/urdf/ip_bh280.urdf.xacro (robot description, xacro)
@@ -2,5 +2,7 @@
 <robot xmlns:xacro="http://ros.org/wiki/xacro">
 	<!-- Import all Gazebo-customization elements, including Gazebo colors -->
-	<xacro:include filename="$(find barrett_hand_description)/urdf/bh282.gazebo.xacro" />
+	<xacro:include filename="$(find barrett_hand_description)/urdf/ip_bh280.gazebo.xacro" />
+	<!-- Import all transmissions -->
+	<xacro:include filename="$(find barrett_hand_description)/urdf/ip_bh280.transmission.xacro" />
 	<!-- Constants for robot dimensions -->
 	<xacro:property name="PI" value="3.1415926535897931"/>
@@ -10,6 +12,5 @@
 	<xacro:property name="joint_effort_limit" value="30.0" />
 	<xacro:property name="joint_velocity_limit" value="2.0" />
-	<xacro:property name="mechanical_reduction" value="1.0" />
-	<xacro:macro name="bhand_macro" params="parent name *origin">
+	<xacro:macro name="bhand_macro" params="parent name namespace *origin">
         <!-- base joint (FIXED) -->
 		<joint name="${name}_base_joint" type="fixed">
@@ -42,90 +43,4 @@
 			</collision>
 		</link>
-		<!-- finger 3 -->
-		<!-- finger 32 link -->
-		<link name="${name}_finger_32_link">
-			 <inertial>
-				<mass value="0.1"/>
-				<origin xyz="0 0 0" rpy="0 0 0"/>
-				<inertia ixx="0.01" ixy="0" ixz="0" iyy="0.01" iyz="0" izz="0.01" />
-			 </inertial>
-			 <visual>
-				<origin xyz="0 0 0" rpy="0 0 0" />
-				<geometry>
-				  <mesh filename="package://barrett_hand_description/meshes/finger.dae" />
-				</geometry>
-				<material name="Blue" />
-			 </visual>
-			 <collision>
-				<origin xyz="0 0 0" rpy="0 0 0" />
-				<geometry>
-				  <mesh filename="package://barrett_hand_description/meshes/finger.dae" />
-				</geometry>
-				<contact_coefficients kd="1.0" kp="1000.0" mu="0"/>
-			 </collision>
-		</link>
-		<!-- joint 32 between BH_base_link (PALM) and BH_finger_32_link -->
-		<joint name="${name}_j32_joint" type="revolute">
-			<parent link="${name}_base_link"/>
-			<child link="${name}_finger_32_link"/>
-			<origin xyz="0 -0.05 0.0754" rpy="1.5708 0 1.5708" />
-			<axis xyz="0 0 -1"/>
-			<limit effort="${joint_effort_limit}" lower="0.0" upper="2.44" velocity="${joint_velocity_limit}"/>
-			<dynamics damping="${joint_damping}" friction="${joint_friction}"/>
-		</joint>
-		<transmission name="${name}_j32_transmission">
-			<type>transmission_interface/SimpleTransmission</type>
-			<joint name="${name}_j32_joint">
-			  <hardwareInterface>hardware_interface/PositionJointInterface</hardwareInterface>
-			</joint>
-			<actuator name="${name}_j32">
-			  <hardwareInterface>hardware_interface/PositionJointInterface</hardwareInterface>
-			  <mechanicalReduction>1</mechanicalReduction>
-			  <motorTorqueConstant>1</motorTorqueConstant>
-			</actuator>
-		</transmission>
-		<!-- finger 33 link -->
-		<link name="${name}_finger_33_link">
-		 <inertial>
-			<mass value="0.1"/>
-			<origin xyz="0 0 0" rpy="0 0 0"/>
-			<inertia ixx="0.01" ixy="0" ixz="0" iyy="0.01" iyz="0" izz="0.01" />
-		 </inertial>
-		 <visual>
-			<origin xyz="0 0 0" rpy="0 0 0" />
-			<geometry>
-			  <mesh filename="package://barrett_hand_description/meshes/finger_tip.dae" />
-			</geometry>
-			<material name="Blue" />
-		 </visual>
-		 <collision>
-			<origin xyz="0 0 0" rpy="0 0 0" />
-			<geometry>
-			  <mesh filename="package://barrett_hand_description/meshes/finger_tip.dae" />
-			</geometry>
-			<contact_coefficients kd="1.0" kp="1000.0" mu="0"/>
-		 </collision>
-		</link>
-		<!-- joint 33 between BH_finger_32_link and BH_finger_33_link -->
-		<joint name="${name}_j33_joint" type="revolute">
-			<parent link="${name}_finger_32_link"/>
-			<child link="${name}_finger_33_link"/>
-			<origin xyz="-0.069936 0.003 0" rpy="0 0 0" />
-			<axis xyz="0 0 -1"/>
-			<mimic joint="${name}_j32_joint" multiplier="${0.84/2.44}" />
-			<limit effort="${joint_effort_limit}" lower="0.0" upper="0.84" velocity="${joint_velocity_limit}"/>
-			<dynamics damping="${joint_damping}" friction="${joint_friction}"/>
-		</joint>
-		<transmission name="${name}_j33_transmission">
-			<type>transmission_interface/SimpleTransmission</type>
-			<joint name="${name}_j33_joint">
- 			   <hardwareInterface>hardware_interface/PositionJointInterface</hardwareInterface>
-			</joint>
-			<actuator name="${name}_j33">
-			  <hardwareInterface>hardware_interface/PositionJointInterface</hardwareInterface>
-			  <mechanicalReduction>1</mechanicalReduction>
-			  <motorTorqueConstant>1</motorTorqueConstant>
-			</actuator>
-		</transmission>
 		<!-- finger 1 -->
 		<!-- finger 11 link (KNUCKLE) -->
@@ -159,15 +74,4 @@
 			<dynamics damping="${joint_damping}" friction="${joint_friction}"/>
 		</joint>
-		<transmission name="${name}_j11_transmission">
-			<type>transmission_interface/SimpleTransmission</type>
-			<joint name="${name}_j11_joint">
-			   <hardwareInterface>hardware_interface/PositionJointInterface</hardwareInterface>
-			</joint>
-			<actuator name="${name}_j11">
-			  <hardwareInterface>hardware_interface/PositionJointInterface</hardwareInterface>
-			  <mechanicalReduction>1</mechanicalReduction>
-			  <motorTorqueConstant>1</motorTorqueConstant>
-			</actuator>
-		</transmission>
 		<!-- finger 12 link (FINGER) -->
 		<link name="${name}_finger_12_link">
@@ -202,15 +106,4 @@
 			<dynamics damping="${joint_damping}" friction="${joint_friction}"/>
 		</joint>
-		<transmission name="${name}_j12_transmission">
-			<type>transmission_interface/SimpleTransmission</type>
-			<joint name="${name}_j12_joint">
-			   <hardwareInterface>hardware_interface/PositionJointInterface</hardwareInterface>
-			</joint>
-			<actuator name="${name}_j12">
-			  <hardwareInterface>hardware_interface/PositionJointInterface</hardwareInterface>
-			  <mechanicalReduction>1</mechanicalReduction>
-			  <motorTorqueConstant>1</motorTorqueConstant>
-			</actuator>
-		</transmission>
 		<!-- finger 13 link (FINGER TIP) -->
 		<link name="${name}_finger_13_link">
@@ -241,19 +134,8 @@
 			<origin xyz="-0.069936 0.003 0" rpy="0 0 0" />
 			<axis xyz="0 0 -1"/>
-			<mimic joint="${name}_j12_joint" multiplier="${0.84/2.44}" />
+			<!--<mimic joint="${name}_j12_joint" multiplier="${0.84/2.44}" />-->
 			<limit effort="${joint_effort_limit}" lower="0.0" upper="0.84" velocity="${joint_velocity_limit}"/>
 			<dynamics damping="${joint_damping}" friction="${joint_friction}"/>
 		</joint>
-		<transmission name="${name}_j13_transmission">
-			<type>transmission_interface/SimpleTransmission</type>
-			<joint name="${name}_j13_joint">
-			   <hardwareInterface>hardware_interface/PositionJointInterface</hardwareInterface>
-			</joint>
-			<actuator name="${name}_j13">
-			  <hardwareInterface>hardware_interface/PositionJointInterface</hardwareInterface>
-			  <mechanicalReduction>1</mechanicalReduction>
-			  <motorTorqueConstant>1</motorTorqueConstant>
-			</actuator>
-		</transmission>
 		<!-- finger 2 -->
 		<!-- finger 21 link (KNUCKLE) -->
@@ -284,19 +166,8 @@
 			<origin xyz="-0.025 0 0.0415" rpy="0 0 -1.5708" />
 			<axis xyz="0 0 1"/>
-			<mimic joint="${name}_j11_joint" multiplier="1" />
+			<!--<mimic joint="${name}_j11_joint" multiplier="1" />-->
 			<limit effort="${joint_effort_limit}" lower="0" upper="3.1416" velocity="${joint_velocity_limit}"/>
 			<dynamics damping="${joint_damping}" friction="${joint_friction}"/>
 		</joint>
-		<transmission name="${name}_j21_transmission">
-			<type>transmission_interface/SimpleTransmission</type>
-			<joint name="${name}_j21_joint">
-			   <hardwareInterface>hardware_interface/PositionJointInterface</hardwareInterface>
-			</joint>
-			<actuator name="${name}_j21">
-			  <hardwareInterface>hardware_interface/PositionJointInterface</hardwareInterface>
-			  <mechanicalReduction>1</mechanicalReduction>
-			  <motorTorqueConstant>1</motorTorqueConstant>
-			</actuator>
-		</transmission>
 		<!-- finger 22 link (FINGER) -->
 		<link name="${name}_finger_22_link">
@@ -331,15 +202,4 @@
 			<dynamics damping="${joint_damping}" friction="${joint_friction}"/>
 		</joint>
-		<transmission name="${name}_j22_transmission">
-			<type>transmission_interface/SimpleTransmission</type>
-			<joint name="${name}_j22_joint">
- 			   <hardwareInterface>hardware_interface/PositionJointInterface</hardwareInterface>
-			</joint>
-			<actuator name="${name}_j22">
-			  <hardwareInterface>hardware_interface/PositionJointInterface</hardwareInterface>
-			  <mechanicalReduction>1</mechanicalReduction>
-			  <motorTorqueConstant>1</motorTorqueConstant>
-			</actuator>
-		</transmission>
 		<!-- finger 23 link (FINGER TIP) -->
 		<link name="${name}_finger_23_link">
@@ -370,20 +230,74 @@
 			<origin xyz="-0.069936 0.003 0" rpy="0 0 0" />
 			<axis xyz="0 0 -1"/>
-			<mimic joint="${name}_j22_joint" multiplier="${0.84/2.44}" />
+			<!--<mimic joint="${name}_j22_joint" multiplier="${0.84/2.44}" />-->
 			<limit effort="${joint_effort_limit}" lower="0.0" upper="0.84" velocity="${joint_velocity_limit}"/>
 			<dynamics damping="${joint_damping}" friction="${joint_friction}"/>
 		</joint>
-		<transmission name="${name}_j23_transmission">
-			<type>transmission_interface/SimpleTransmission</type>
-			<joint name="${name}_j23_joint">
-			   <hardwareInterface>hardware_interface/PositionJointInterface</hardwareInterface>
-			</joint>
-			<actuator name="${name}_j23">
-			  <hardwareInterface>hardware_interface/PositionJointInterface</hardwareInterface>
-			  <mechanicalReduction>1</mechanicalReduction>
-			  <motorTorqueConstant>1</motorTorqueConstant>
-			</actuator>
-		</transmission>
-		<xacro:bh_gazebo name="${name}"/>
+		<!-- finger 3 -->
+		<!-- finger 32 link -->
+		<link name="${name}_finger_32_link">
+			 <inertial>
+				<mass value="0.1"/>
+				<origin xyz="0 0 0" rpy="0 0 0"/>
+				<inertia ixx="0.01" ixy="0" ixz="0" iyy="0.01" iyz="0" izz="0.01" />
+			 </inertial>
+			 <visual>
+				<origin xyz="0 0 0" rpy="0 0 0" />
+				<geometry>
+				  <mesh filename="package://barrett_hand_description/meshes/finger.dae" />
+				</geometry>
+				<material name="Blue" />
+			 </visual>
+			 <collision>
+				<origin xyz="0 0 0" rpy="0 0 0" />
+				<geometry>
+				  <mesh filename="package://barrett_hand_description/meshes/finger.dae" />
+				</geometry>
+				<contact_coefficients kd="1.0" kp="1000.0" mu="0"/>
+			 </collision>
+		</link>
+		<!-- joint 32 between BH_base_link (PALM) and BH_finger_32_link -->
+		<joint name="${name}_j32_joint" type="revolute">
+			<parent link="${name}_base_link"/>
+			<child link="${name}_finger_32_link"/>
+			<origin xyz="0 -0.05 0.0754" rpy="1.5708 0 1.5708" />
+			<axis xyz="0 0 -1"/>
+			<limit effort="${joint_effort_limit}" lower="0.0" upper="2.44" velocity="${joint_velocity_limit}"/>
+			<dynamics damping="${joint_damping}" friction="${joint_friction}"/>
+		</joint>
+		<!-- finger 33 link -->
+		<link name="${name}_finger_33_link">
+		 <inertial>
+			<mass value="0.1"/>
+			<origin xyz="0 0 0" rpy="0 0 0"/>
+			<inertia ixx="0.01" ixy="0" ixz="0" iyy="0.01" iyz="0" izz="0.01" />
+		 </inertial>
+		 <visual>
+			<origin xyz="0 0 0" rpy="0 0 0" />
+			<geometry>
+			  <mesh filename="package://barrett_hand_description/meshes/finger_tip.dae" />
+			</geometry>
+			<material name="Blue" />
+		 </visual>
+		 <collision>
+			<origin xyz="0 0 0" rpy="0 0 0" />
+			<geometry>
+			  <mesh filename="package://barrett_hand_description/meshes/finger_tip.dae" />
+			</geometry>
+			<contact_coefficients kd="1.0" kp="1000.0" mu="0"/>
+		 </collision>
+		</link>
+		<!-- joint 33 between BH_finger_32_link and BH_finger_33_link -->
+		<joint name="${name}_j33_joint" type="revolute">
+			<parent link="${name}_finger_32_link"/>
+			<child link="${name}_finger_33_link"/>
+			<origin xyz="-0.069936 0.003 0" rpy="0 0 0" />
+			<axis xyz="0 0 -1"/>
+			<!--<mimic joint="${name}_j32_joint" multiplier="${0.84/2.44}" />-->
+			<limit effort="${joint_effort_limit}" lower="0.0" upper="0.84" velocity="${joint_velocity_limit}"/>
+			<dynamics damping="${joint_damping}" friction="${joint_friction}"/>
+		</joint>
+		<xacro:bh280_transmission name="${name}"/>
+		<xacro:bh_gazebo name="${name}" namespace="${namespace}"/>
 	</xacro:macro>
 </robot>
