Commit message: Adding contact to barrett hand

File: effectors/barrett_hand/barrett_hand_common/barrett_hand_description/urdf/ip_bh280.gazebo.xacro (robot description, xacro)
@@ -8,43 +8,215 @@
 	</gazebo>
 	<gazebo reference="${name}_base_link">
+		  <sensor type="contact" name="${name}_base_link_contact">
+			<always_on>1</always_on>
+			<update_rate>1000.0</update_rate>
+			<contact>
+			  <collision>${name}_base_link_geom</collision>
+			  <topic>${name}_base_link_collision</topic>
+			</contact>
+			<plugin name="${name}_palm_gazebo_ros_bumper_controller" filename="libgazebo_ros_bumper.so">
+			  <alwaysOn>true</alwaysOn>
+			  <frameName>${name}_base_link</frameName>
+			  <updateRate>100.0</updateRate>
+			  <bumperTopicName>/contacts/${name}/palm</bumperTopicName>
+			</plugin>
+		  </sensor>
+		  <material>Gazebo/White</material>
+		  <turnGravityOff>False</turnGravityOff>
+	</gazebo>
+	<!--<gazebo reference="${name}_base_link">
 		<material>Gazebo/White</material>
 		<turnGravityOff>False</turnGravityOff>
-	</gazebo>
-	<gazebo reference="${name}_finger_31_link">
-		<material>Gazebo/Grey</material>
-		<turnGravityOff>False</turnGravityOff>
-	</gazebo>
+	</gazebo>-->
+	<gazebo reference="${name}_finger_11_link">
+		  <sensor type="contact" name="${name}_finger_11_link_contact">
+			<always_on>1</always_on>
+			<update_rate>1000.0</update_rate>
+			<contact>
+			  <collision>${name}_finger_11_link_geom</collision>
+			  <topic>${name}_finger_11_link_collision</topic>
+			</contact>
+			<plugin name="${name}_finger1_knuckle_gazebo_ros_bumper_controller" filename="libgazebo_ros_bumper.so">
+			  <alwaysOn>true</alwaysOn>
+			  <frameName>${name}_finger_11_link</frameName>
+			  <updateRate>100.0</updateRate>
+			  <bumperTopicName>/contacts/${name}/finger1/knuckle</bumperTopicName>
+			</plugin>
+		  </sensor>
+		  <selfCollide>false</selfCollide>
+		  <material>Gazebo/Grey</material>
+		  <turnGravityOff>False</turnGravityOff>
+	</gazebo>
+	<!--<gazebo reference="${name}_finger_11_link">
+		<material>Gazebo/Grey</material>
+		<turnGravityOff>False</turnGravityOff>
+	</gazebo>-->
+	<gazebo reference="${name}_finger_12_link">
+		  <sensor type="contact" name="${name}_finger_12_link_contact">
+			<always_on>1</always_on>
+			<update_rate>1000.0</update_rate>
+			<contact>
+			  <collision>${name}_finger_12_link_geom</collision>
+			  <topic>${name}_finger_12_link_collision</topic>
+			</contact>
+			<plugin name="${name}_finger1_proximal_gazebo_ros_bumper_controller" filename="libgazebo_ros_bumper.so">
+			  <alwaysOn>true</alwaysOn>
+			  <frameName>${name}_finger_12_link</frameName>
+			  <updateRate>100.0</updateRate>
+			  <bumperTopicName>/contacts/${name}/finger1/proximal</bumperTopicName>
+			</plugin>
+		  </sensor>
+		  <selfCollide>false</selfCollide>
+		  <material>Gazebo/Grey</material>
+		  <turnGravityOff>False</turnGravityOff>
+		  <selfCollide>true</selfCollide>
+	</gazebo>
+	<!--<gazebo reference="${name}_finger_12_link">
+		<material>Gazebo/Grey</material>
+		<turnGravityOff>False</turnGravityOff>
+	</gazebo>-->
+	<gazebo reference="${name}_finger_13_link">
+		  <sensor type="contact" name="${name}_finger_13_link_contact">
+			<always_on>1</always_on>
+			<update_rate>1000.0</update_rate>
+			<contact>
+			  <collision>${name}_finger_13_link_geom</collision>
+			  <topic>${name}_finger_13_link_collision</topic>
+			</contact>
+			<plugin name="${name}_finger1_distal_gazebo_ros_bumper_controller" filename="libgazebo_ros_bumper.so">
+			  <alwaysOn>true</alwaysOn>
+			  <frameName>${name}_finger_13_link</frameName>
+			  <updateRate>100.0</updateRate>
+			  <bumperTopicName>/contacts/${name}/finger1/distal</bumperTopicName>
+			</plugin>
+		  </sensor>
+		  <selfCollide>false</selfCollide>
+		  <material>Gazebo/Grey</material>
+		  <turnGravityOff>False</turnGravityOff>
+		  <selfCollide>true</selfCollide>
+	</gazebo>
+	<!--<gazebo reference="${name}_finger_13_link">
+		<material>Gazebo/Grey</material>
+		<turnGravityOff>False</turnGravityOff>
+	</gazebo>-->
+	<gazebo reference="${name}_finger_21_link">
+		  <sensor type="contact" name="${name}_finger_21_link_contact">
+			<always_on>1</always_on>
+			<update_rate>1000.0</update_rate>
+			<contact>
+			  <collision>${name}_finger_21_link_geom</collision>
+			  <topic>${name}_finger_21_link_collision</topic>
+			</contact>
+			<plugin name="${name}_finger2_knuckle_gazebo_ros_bumper_controller" filename="libgazebo_ros_bumper.so">
+			  <alwaysOn>true</alwaysOn>
+			  <frameName>${name}_finger_21_link</frameName>
+			  <updateRate>100.0</updateRate>
+			  <bumperTopicName>/contacts/${name}/finger2/knuckle</bumperTopicName>
+			</plugin>
+		  </sensor>
+		  <selfCollide>false</selfCollide>
+		  <material>Gazebo/Grey</material>
+		  <turnGravityOff>False</turnGravityOff>
+	</gazebo>
+	<!--<gazebo reference="${name}_finger_21_link">
+		<material>Gazebo/Grey</material>
+		<turnGravityOff>False</turnGravityOff>
+	</gazebo>-->
+	<gazebo reference="${name}_finger_22_link">
+		  <sensor type="contact" name="${name}_finger_22_link_contact">
+			<always_on>1</always_on>
+			<update_rate>1000.0</update_rate>
+			<contact>
+			  <collision>${name}_finger_22_link_geom</collision>
+			  <topic>${name}_finger_22_link_collision</topic>
+			</contact>
+			<plugin name="${name}_finger2_proximal_gazebo_ros_bumper_controller" filename="libgazebo_ros_bumper.so">
+			  <alwaysOn>true</alwaysOn>
+			  <frameName>${name}_finger_22_link</frameName>
+			  <updateRate>100.0</updateRate>
+			  <bumperTopicName>/contacts/${name}/finger2/proximal</bumperTopicName>
+			</plugin>
+		  </sensor>
+		  <selfCollide>false</selfCollide>
+		  <material>Gazebo/Grey</material>
+		  <turnGravityOff>False</turnGravityOff>
+		  <selfCollide>true</selfCollide>
+	</gazebo>
+	<!--<gazebo reference="${name}_finger_22_link">
+		<material>Gazebo/Grey</material>
+		<turnGravityOff>False</turnGravityOff>
+	</gazebo>-->
+	<gazebo reference="${name}_finger_23_link">
+		  <sensor type="contact" name="${name}_finger_23_link_contact">
+			<always_on>1</always_on>
+			<update_rate>1000.0</update_rate>
+			<contact>
+			  <collision>${name}_finger_23_link_geom</collision>
+			  <topic>${name}_finger_23_link_collision</topic>
+			</contact>
+			<plugin name="${name}_finger2_distal_gazebo_ros_bumper_controller" filename="libgazebo_ros_bumper.so">
+			  <alwaysOn>true</alwaysOn>
+			  <frameName>${name}_finger_23_link</frameName>
+			  <updateRate>100.0</updateRate>
+			  <bumperTopicName>/contacts/${name}/finger2/distal</bumperTopicName>
+			</plugin>
+		  </sensor>
+		  <selfCollide>false</selfCollide>
+		  <material>Gazebo/Grey</material>
+		  <turnGravityOff>False</turnGravityOff>
+		  <selfCollide>true</selfCollide>
+	</gazebo>
+	<!--<gazebo reference="${name}_finger_23_link">
+		<material>Gazebo/Grey</material>
+		<turnGravityOff>False</turnGravityOff>
+	</gazebo>-->
 	<gazebo reference="${name}_finger_32_link">
-		<material>Gazebo/Grey</material>
-		<turnGravityOff>False</turnGravityOff>
-	</gazebo>
+		  <sensor type="contact" name="${name}_finger_32_link_contact">
+			<always_on>1</always_on>
+			<update_rate>1000.0</update_rate>
+			<contact>
+			  <collision>${name}_finger_32_link_geom</collision>
+			  <topic>${name}_finger_32_link_collision</topic>
+			</contact>
+			<plugin name="${name}_finger3_proximal_gazebo_ros_bumper_controller" filename="libgazebo_ros_bumper.so">
+			  <alwaysOn>true</alwaysOn>
+			  <frameName>${name}_finger_32_link</frameName>
+			  <updateRate>100.0</updateRate>
+			  <bumperTopicName>/contacts/${name}/finger3/proximal</bumperTopicName>
+			</plugin>
+		  </sensor>
+		  <selfCollide>false</selfCollide>
+		  <material>Gazebo/Grey</material>
+		  <turnGravityOff>False</turnGravityOff>
+		  <selfCollide>true</selfCollide>
+	</gazebo>
+	<!--<gazebo reference="${name}_finger_32_link">
+		<material>Gazebo/Grey</material>
+		<turnGravityOff>False</turnGravityOff>
+	</gazebo>-->
 	<gazebo reference="${name}_finger_33_link">
-		<material>Gazebo/Grey</material>
-		<turnGravityOff>False</turnGravityOff>
-	</gazebo>
-	<gazebo reference="${name}_finger_11_link">
-		<material>Gazebo/Grey</material>
-		<turnGravityOff>False</turnGravityOff>
-	</gazebo>
-	<gazebo reference="${name}_finger_12_link">
-		<material>Gazebo/Grey</material>
-		<turnGravityOff>False</turnGravityOff>
-	</gazebo>
-	<gazebo reference="${name}_finger_13_link">
-		<material>Gazebo/Grey</material>
-		<turnGravityOff>False</turnGravityOff>
-	</gazebo>
-	<gazebo reference="${name}_finger_21_link">
-		<material>Gazebo/Grey</material>
-		<turnGravityOff>False</turnGravityOff>
-	</gazebo>
-	<gazebo reference="${name}_finger_22_link">
-		<material>Gazebo/Grey</material>
-		<turnGravityOff>False</turnGravityOff>
-	</gazebo>
-	<gazebo reference="${name}_finger_23_link">
-		<material>Gazebo/Grey</material>
-		<turnGravityOff>False</turnGravityOff>
-	</gazebo>
+		  <sensor type="contact" name="${name}_finger_33_link_contact">
+			<always_on>1</always_on>
+			<update_rate>1000.0</update_rate>
+			<contact>
+			  <collision>${name}_finger_33_link_geom</collision>
+			  <topic>${name}_finger_33_link_collision</topic>
+			</contact>
+			<plugin name="${name}_finger3_distal_gazebo_ros_bumper_controller" filename="libgazebo_ros_bumper.so">
+			  <alwaysOn>true</alwaysOn>
+			  <frameName>${name}_finger_33_link</frameName>
+			  <updateRate>100.0</updateRate>
+			  <bumperTopicName>/contacts/${name}/finger3/distal</bumperTopicName>
+			</plugin>
+		  </sensor>
+		  <selfCollide>false</selfCollide>
+		  <material>Gazebo/Grey</material>
+		  <turnGravityOff>False</turnGravityOff>
+		  <selfCollide>true</selfCollide>
+	</gazebo>
+	<!--<gazebo reference="${name}_finger_33_link">
+		<material>Gazebo/Grey</material>
+		<turnGravityOff>False</turnGravityOff>
+	</gazebo>-->
   </xacro:macro>
 </robot>

File: effectors/barrett_hand/barrett_hand_common/barrett_hand_description/urdf/ip_bh280.urdf.xacro (robot description, xacro)
@@ -37,5 +37,5 @@
 			<collision>
 			   <origin xyz="0 0 0" rpy="0 0 0 " />
-			   <geometry>
+			   <geometry name="${name}_base_link_geom">
 				  <mesh filename="package://barrett_hand_description/meshes/palm_280.dae"/>
 			   </geometry>
@@ -60,5 +60,5 @@
 			<collision>
 			  <origin xyz="0 0 0" rpy="0 0 0" />
-			  <geometry>
+			  <geometry name="${name}_finger_11_link_geom">
 				<mesh filename="package://barrett_hand_description/meshes/knuckle.dae" />
 			  </geometry>
@@ -74,5 +74,5 @@
 			<dynamics damping="${joint_damping}" friction="${joint_friction}"/>
 		</joint>
-		<!-- finger 12 link (FINGER) -->
+		<!-- finger 12 link (FINGER) (PROXIMAL) -->
 		<link name="${name}_finger_12_link">
 			 <inertial>
@@ -90,5 +90,5 @@
 			 <collision>
 				<origin xyz="0 0 0" rpy="0 0 0" />
-				<geometry>
+				<geometry name="${name}_finger_12_link_geom">
 				  <mesh filename="package://barrett_hand_description/meshes/finger.dae" />
 				</geometry>
@@ -106,5 +106,5 @@
 			<dynamics damping="${joint_damping}" friction="${joint_friction}"/>
 		</joint>
-		<!-- finger 13 link (FINGER TIP) -->
+		<!-- finger 13 link (FINGER TIP) (DISTAL) -->
 		<link name="${name}_finger_13_link">
 		 <inertial>
@@ -122,5 +122,5 @@
 		 <collision>
 			<origin xyz="0 0 0" rpy="0 0 0" />
-			<geometry>
+			<geometry name="${name}_finger_13_link_geom">
 			  <mesh filename="package://barrett_hand_description/meshes/finger_tip.dae" />
 			</geometry>
@@ -155,5 +155,5 @@
 			<collision>
 			  <origin xyz="0 0 0" rpy="0 0 0" />
-			  <geometry>
+			  <geometry name="${name}_finger_21_link_geom">
 				<mesh filename="package://barrett_hand_description/meshes/knuckle.dae" />
 			  </geometry>
@@ -170,5 +170,5 @@
 			<dynamics damping="${joint_damping}" friction="${joint_friction}"/>
 		</joint>
-		<!-- finger 22 link (FINGER) -->
+		<!-- finger 22 link (FINGER) (PROXIMAL) -->
 		<link name="${name}_finger_22_link">
 			 <inertial>
@@ -186,5 +186,5 @@
 			 <collision>
 				<origin xyz="0 0 0" rpy="0 0 0" />
-				<geometry>
+				<geometry name="${name}_finger_22_link_geom">
 				  <mesh filename="package://barrett_hand_description/meshes/finger.dae" />
 				</geometry>
@@ -202,5 +202,5 @@
 			<dynamics damping="${joint_damping}" friction="${joint_friction}"/>
 		</joint>
-		<!-- finger 23 link (FINGER TIP) -->
+		<!-- finger 23 link (FINGER TIP) (DISTAL) -->
 		<link name="${name}_finger_23_link">
 		 <inertial>
@@ -218,5 +218,5 @@
 		 <collision>
 			<origin xyz="0 0 0" rpy="0 0 0" />
-			<geometry>
+			<geometry name="${name}_finger_23_link_geom">
 			  <mesh filename="package://barrett_hand_description/meshes/finger_tip.dae" />
 			</geometry>
@@ -235,5 +235,5 @@
 		</joint>
 		<!-- finger 3 -->
-		<!-- finger 32 link -->
+		<!-- finger 32 link (PROXIMAL) -->
 		<link name="${name}_finger_32_link">
 			 <inertial>
@@ -251,5 +251,5 @@
 			 <collision>
 				<origin xyz="0 0 0" rpy="0 0 0" />
-				<geometry>
+				<geometry name="${name}_finger_32_link_geom">
 				  <mesh filename="package://barrett_hand_description/meshes/finger.dae" />
 				</geometry>
@@ -266,5 +266,5 @@
 			<dynamics damping="${joint_damping}" friction="${joint_friction}"/>
 		</joint>
-		<!-- finger 33 link -->
+		<!-- finger 33 link (DISTAL) -->
 		<link name="${name}_finger_33_link">
 		 <inertial>
@@ -282,5 +282,5 @@
 		 <collision>
 			<origin xyz="0 0 0" rpy="0 0 0" />
-			<geometry>
+			<geometry name="${name}_finger_33_link_geom">
 			  <mesh filename="package://barrett_hand_description/meshes/finger_tip.dae" />
 			</geometry>
